File: Right Controller/Budget Joycons (Right).kicad_pcb (KiCad board)
At the start: 4 copper layers, 39.1 x 94.5 mm, 105 parts, among them J1 S2B-PH-K-SLFSN, J2 UJ20-C-H-G-SMT-2A-P16-TR, J3 530480210, J4 PCB Pads, Q1 AO3401A, Q2 AO3401A, Q3 AO3400A, Q4 AO3401A, Q5 AO3401A, Q6 AO3400A, SW1 B3F_1020, SW10 SKSCLBE010, SW11 SKSCLBE010, SW12 SKSCLBE010, SW2 TL3315NF100Q, SW3 TL3315NF100Q, SW4 TL3315NF100Q, SW5 TL3315NF100Q, SW6 TL3315NF100Q, SW7 TL3315NF100Q, SW8 TL3315NF100Q, SW9 SKSCLBE010, U1 STM32C071CBT6, U2 NRF24L01_Breakout, U3 AP2127K-3.3, U4 MCP73831-2-OT, U5 USBLC6-2SC6, U6 DRV5056A3, U7 DRV5056A3, U8 DRV5056A3, U9 LSM6DSM

Commit message: Right Update
Routing:
- net +3.3V: track 138.5 -> 247.9 mm, vias 10 -> 14
- net POWER_BUTTON: track 2.77 -> 94.2 mm, vias 0 -> 3
- net GND: track 98.4 -> 187.1 mm, vias 25 -> 52
- net RUMBLE_ENABLE: track 0.00 -> 64.2 mm, vias 0 -> 2
- net +3.3V SIDE TRIGGERS: track 4.35 -> 62.7 mm, vias 0 -> 2
- net ANALOG_JOYSTICK_X: track 1.67 -> 44.7 mm, vias 0 -> 3
- net Net-(U6-OUT): track 0.00 -> 37.5 mm, vias 0 -> 2
- net ANALOG_JOYSTICK_Y: track 1.67 -> 34.7 mm, vias 0 -> 1
- net POWER_HOLD: track 0.00 -> 31.7 mm, vias 0 -> 3
- net TRIGGER_MODE_SIDE: track 0.99 -> 26.0 mm, vias 0 -> 3
- net TRIGGER_MODE_MAIN: track 0.00 -> 22.6 mm
- net +VSYS: track 8.01 -> 29.2 mm, vias 0 -> 1
- net Net-(D5-K): track 0.00 -> 19.7 mm, vias 0 -> 4
- net IMU_IRQ2: track 0.00 -> 19.1 mm, vias 0 -> 1
- net IMU_IRQ1: track 0.00 -> 12.8 mm, vias 0 -> 1
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- added copper zone on In1.Cu, net +3.3V
- added copper zone on In1.Cu, net Net-(D5-K)

Commit message: Further Right Side Updates
Parts:
- moved R5 0.35 mm to (140.5, 74.7)
- moved R3 0.26 mm to (139.3, 75.9)
Routing:
- net Net-(Q3-G): track 13.2 -> 77.9 mm, vias 1 -> 3
- net +3.3V: track 247.9 -> 303.9 mm, vias 14 -> 18
- net BUTTON_BUMPER_MAIN: track 6.56 -> 56.4 mm, vias 0 -> 2
- net +VSYS: track 29.2 -> 74.2 mm, vias 1 -> 3
- net Net-(U8-OUT): track 0.00 -> 44.5 mm, vias 0 -> 2
- net BUTTON_EXTRA_3: track 8.55 -> 51.6 mm, vias 2 -> 4
- net BUTTON_LEFT: track 0.00 -> 36.5 mm, vias 0 -> 4
- net BUTTON_BUMPER_RIGHT: track 2.93 -> 37.8 mm, vias 1 -> 2
- net BUTTON_DOWN: track 4.46 -> 33.2 mm, vias 0 -> 3
- net +5V: track 46.1 -> 69.4 mm, vias 3 -> 5
- net I2C_IMU_SCL: track 1.77 -> 24.6 mm, vias 0 -> 2
- net BUTTON_UP: track 4.46 -> 26.4 mm, vias 0 -> 3
- net I2C_IMU_SDA: track 2.20 -> 15.7 mm, vias 0 -> 1
- net BUTTON_RIGHT: track 4.46 -> 14.9 mm, vias 0 -> 1
- net GND: track 187.1 -> 193.8 mm
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
Commit message: Pre DRC right upload
Routing:
- net LED_1: track 2.48 -> 65.0 mm, vias 1 -> 3
- net LED_0: track 2.25 -> 61.5 mm, vias 1 -> 4
- net ANALOG_BATT: track 1.76 -> 51.6 mm, vias 0 -> 3
- net LED_3: track 1.50 -> 40.8 mm, vias 1 -> 2
- net BUTTON_UP: track 26.4 -> 59.9 mm, vias 3 -> 4
- net BUTTON_RIGHT: track 14.9 -> 47.5 mm, vias 1 -> 2
- net LED_2: track 2.45 -> 33.3 mm, vias 1 -> 2
- net +VBAT: track 9.88 -> 37.7 mm, vias 0 -> 2
- net +3.3V: track 303.9 -> 310.8 mm, vias 18 -> 19
- net Net-(D8-K): track 0.00 -> 2.42 mm, vias 0 -> 1
- net TRIGGER_MODE_MAIN: track 22.6 -> 24.0 mm
- net BUTTON_LEFT: track 36.5 -> 37.8 mm
- net ANALOG_JOYSTICK_Y: track 34.3 -> 33.5 mm
- net +VSYS: track 74.2 -> 73.4 mm
- net BUTTON_BUMPER_MAIN: track 56.4 -> 55.6 mm
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